Commit message: Done: Task1

File: my_rb1_description/urdf/my_rb1_robot.urdf (robot description, URDF)
Before this commit: robot robot, 7 links, 6 joints
Joints:
- joint base_footprint_base_link_joint: origin xyz=0 0 0 rpy=0 0 0 -> xyz=0 0 0.20 rpy=0 0 0

Commit message: Change: base_footprint pos

File: my_rb1_description/urdf/my_rb1_robot.urdf (robot description, URDF)
Before this commit: robot robot, 7 links, 6 joints
Links:
- link front_laser: geometry collision cylinder length=0.10 radius=0.05; visual cylinder length=0.04 radius=0.02
Joints:
- removed joint base_footprint_base_link_joint
- added joint base_link_base_footprint_joint: type fixed, parent base_footprint, child base_link, origin xyz=0 0 0.15 rpy=0 0 0

Commit message: Change: wheel params

File: my_rb1_description/urdf/my_rb1_robot.urdf (robot description, URDF)
Before this commit: robot robot, 7 links, 6 joints
Links:
- link left_wheel: mass 2.125 -> 1
- link right_wheel: mass 2.125 -> 1
Joints:
- joint base_link_left_wheel_joint: limit effort=10000 velocity=1000 -> (none); origin xyz=0 0.2 -0.15 rpy=0 0 0 -> xyz=0 0.2 -0.15 rpy=0 -1.5708 0
- joint base_link_right_wheel_joint: limit effort=10000 velocity=1000 -> (none); origin xyz=0 -0.2 -0.15 rpy=0 0 0 -> xyz=0 -0.2 -0.15 rpy=0 -1.5708 0
